File: GBA_lipo/_autosave-GBA_lipo.kicad_sch (KiCad schematic)
At the start: 33 parts, among them J1 USB_C_Receptacle, J2 BATT CONN, J3 Conn_01x02_Female, U1 AMS1117-1.5, U2 TP4056-42-ESOP8, U3 LM393, U4 B5819W SL, U5 WTM3401, U6 NCP1529, U7 2N7002_

Commit message: Layout work
Parts:
- gave numbers to parts that had none: 2
Changed lines of the file:
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@@
   (symbol (lib_id "Device:LED") (at 80.01 39.37 90) (unit 1)
     (in_bom yes) (on_board yes)
-    (property "Reference" "D?" (id 0) (at 77.47 38.1 0)
+    (property "Reference" "D1" (id 0) (at 77.47 38.1 0)
       (effects (font (size 1.27 1.27)) (justify right))
     )
@@
   (symbol (lib_id "Device:LED") (at 88.9 39.37 90) (unit 1)
     (in_bom yes) (on_board yes)
-    (property "Reference" "D?" (id 0) (at 86.36 38.1 0)
+    (property "Reference" "D2" (id 0) (at 86.36 38.1 0)
       (effects (font (size 1.27 1.27)) (justify right))
     )
@@
     )
     (path "/0022ecd0-0d5d-43eb-960f-e462c72a9484"
-      (reference "D?") (unit 1) (value "GREEN_LED") (footprint "LED_SMD:LED_0603_1608Metric")
+      (reference "D1") (unit 1) (value "GREEN_LED") (footprint "LED_SMD:LED_0603_1608Metric")
     )
     (path "/eaffb727-c925-4be7-82d6-34c7acf4f871"
-      (reference "D?") (unit 1) (value "RED_LED") (footprint "LED_SMD:LED_0603_1608Metric")
+      (reference "D2") (unit 1) (value "RED_LED") (footprint "LED_SMD:LED_0603_1608Metric")
     )
     (path "/a96882fa-8df4-4031-bf5e-4c4cba60fcaf"
