File: GBA_lipo/GBA_lipo.kicad_pcb (KiCad board)
At the start: 2 copper layers, 40 x 26.1 mm, 32 parts, among them J1 USB_C_Receptacle, J2 BATT CONN, U1 AMS1117-1.5, U2 TP4056-42-ESOP8, U3 LM393, U4 B5819W SL, U5 WTM3401, U6 NCP1529, U7 2N7002_

Commit message: Fab Version 1.0
Parts:
- added G***: LOGO, LOGO, B.Cu at (100.2, 127.0)
- added G***: LOGO, LOGO, B.Cu at (100.0, 127.5)
- added J3: Conn_01x02_Female, Connector_PinHeader_1.27mm:PinHeader_1x02_P1.27mm_Vertical, F.Cu at (117.2, 120.2)
- added JP1: SolderJumper_2_Open, Jumper:SolderJumper-2_P1.3mm_Open_Pad1.0x1.5mm, F.Cu at (108.1, 128.6)
- added JP2: SolderJumper_2_Open, Jumper:SolderJumper-2_P1.3mm_Open_Pad1.0x1.5mm, F.Cu at (106.3, 119.1)
- added JP3: SolderJumper_2_Open, Jumper:SolderJumper-2_P1.3mm_Open_Pad1.0x1.5mm, F.Cu at (104.6, 128.6)
- added JP4: SolderJumper_2_Open, Jumper:SolderJumper-2_P1.3mm_Open_Pad1.0x1.5mm, F.Cu at (101.2, 128.6)
- added JP5: SolderJumper_2_Open, Jumper:SolderJumper-2_P1.3mm_Open_Pad1.0x1.5mm, F.Cu at (87.5, 127.6)
- added R12: 10k, Resistor_SMD:R_0603_1608Metric, F.Cu at (105.7, 124.3)
- added TP1: VDD, TestPoint:TestPoint_Pad_1.0x1.0mm, F.Cu at (107.1, 134.8)
- added TP2: LOW_BATT, TestPoint:TestPoint_Pad_1.0x1.0mm, F.Cu at (105.7, 121.7)
- added TP3: VOUT, TestPoint:TestPoint_Pad_1.0x1.0mm, F.Cu at (117.2, 123.8)
- added TP4: VBAT, TestPoint:TestPoint_Pad_1.0x1.0mm, F.Cu at (83.2, 123.7)
- added TP5: V_SW, TestPoint:TestPoint_Pad_1.0x1.0mm, F.Cu at (107.1, 131.7)
- added TP6: VREF, TestPoint:TestPoint_Pad_1.0x1.0mm, F.Cu at (92.8, 117.0)
- moved R7 119.9 mm to (95.2, 131.4), turned to -90 degrees
- moved U4 111.5 mm to (102.2, 131.7), turned to 180 degrees
- moved U5 110.8 mm to (98.0, 130.9), turned to 90 degrees
- moved R6 91.4 mm to (87.7, 123.3), turned to 180 degrees
- moved RV1 90.8 mm to (87.4, 119.7), turned to 90 degrees
- moved R5 88.4 mm to (87.7, 125.1)
- moved U3 80.9 mm to (92.2, 122.1), turned to -90 degrees
- moved R10 79.2 mm to (111.2, 129.5)
- moved R1 75.5 mm to (108.4, 138.7), turned to -90 degrees
- moved R11 75.1 mm to (111.2, 127.7)
- moved R2 71.3 mm to (106.6, 138.8), turned to -90 degrees
- moved C1 71.2 mm to (103.6, 124.3), turned to 90 degrees
- moved C7 70.8 mm to (114.5, 129.5), turned to 180 degrees
- moved L1 68.0 mm to (113.5, 132.0)
- moved R8 64.3 mm to (109.8, 118.6)
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Connections:
- C1 pad 1: V_SW -> /VI
- C5 pad 2: V_SW -> /VIN
- R5 pad 1: +BATT -> Net-(JP5-A)
- R8 pad 1: LOW_BATT -> Net-(JP2-B)
- U1 pad 3: V_SW -> /VI
- U3 pad 8: V_SW -> /V+
- U6 pad 1: V_SW -> /VIN
- U6 pad 4: V_SW -> /VIN
Routing:
- net GND: track 0.00 -> 28.2 mm, vias 0 -> 8
- net VDD: track 0.00 -> 23.1 mm, vias 0 -> 2
- net LOW_BATT: track 0.00 -> 18.0 mm
- net /V+: track 0.00 -> 15.8 mm, vias 0 -> 2
- net Net-(U6-SW): track 0.00 -> 12.7 mm, vias 0 -> 2
- net Net-(J1-CC1): track 0.00 -> 9.79 mm
- net Net-(U6-FB): track 0.00 -> 9.13 mm
- net Net-(J1-CC2): track 0.00 -> 8.74 mm
- net Net-(U3A-+): track 0.00 -> 6.70 mm
- net Net-(U7-G): track 0.00 -> 6.57 mm
- net Net-(U2-~STDBY): track 0.70 -> 5.81 mm
- net /VI: track 0.00 -> 5.02 mm
- net Net-(U2-PROG): track 0.00 -> 4.76 mm
- net Net-(D1-K): track 0.00 -> 4.20 mm
- net Net-(U2-~CHRG): track 1.08 -> 5.18 mm
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- added copper zone on F.Cu, net +1V5
- added copper zone on F.Cu, net +BATT
- added copper zone on F.Cu, net /VIN
- added copper zone on F.Cu, net GND
- added copper zone on F.Cu, net VDD
- added copper zone on F.Cu, net VOUT
- added copper zone on F.Cu, net V_SW
Other:
- outline, holes or cut-outs redrawn
- board text added: "LITHIUM BOY V1.0"
- board text added: "SEPT 2023"
