File: GBA_lipo/GBA_lipo.kicad_sch (KiCad schematic)
At the start: 33 parts, among them J1 USB_C_Receptacle, J2 BATT CONN, J3 Conn_01x02_Female, U1 AMS1117-1.5, U2 TP4056-42-ESOP8, U3 LM393, U4 B5819W SL, U5 WTM3401, U6 NCP1529, U7 2N7002_

Commit message: Fab Version 1.0
Parts:
- added JP1, JP2, JP3, JP4, JP5: SolderJumper_2_Open, Jumper:SolderJumper-2_P1.3mm_Open_Pad1.0x1.5mm, symbol Jumper:SolderJumper_2_Open
- added R12: 10k, Resistor_SMD:R_0603_1608Metric, symbol Device:R
- added TP1: VDD, TestPoint:TestPoint_Pad_1.0x1.0mm, symbol Connector:TestPoint
- added TP2: LOW_BATT, TestPoint:TestPoint_Pad_1.0x1.0mm, symbol Connector:TestPoint
- added TP3: VOUT, TestPoint:TestPoint_Pad_1.0x1.0mm, symbol Connector:TestPoint
- added TP4: VBAT, TestPoint:TestPoint_Pad_1.0x1.0mm, symbol Connector:TestPoint
- added TP5: V_SW, TestPoint:TestPoint_Pad_1.0x1.0mm, symbol Connector:TestPoint
- added TP6: VREF, TestPoint:TestPoint_Pad_1.0x1.0mm, symbol Connector:TestPoint
- C1, C4: JLCPCB Part # (none) -> C19702; JLC_Part# C19702 -> (none)
- C2: JLCPCB Part # (none) -> C59461; JLC_Part# C59461 -> (none)
- C3: JLCPCB Part # (none) -> C19702; JL_Part# C19702 -> (none)
- J1: JLCPCB Part # (none) -> C709357; JLC_Part# C709357 -> (none)
- J3: footprint (none) -> Connector_PinHeader_1.27mm:PinHeader_1x02_P1.27mm_Vertical
- R1, R2: JLCPCB Part # (none) -> C23186; JLC_Part# C23186 -> (none)
- R3, R4: JLCPCB Part # (none) -> C21190; JLC_Part# C21190 -> (none)
- R5: JLCPCB Part # (none) -> C25197; JLC_Part# C25197 -> (none)
- R6: JLCPCB Part # (none) -> C4260; JLC_Part# C4260 -> (none)
- RPROG1: JLCPCB Part # (none) -> C22843; JLC_Part# C22843 -> (none)
- U1: JLCPCB Part # (none) -> NOT FROM JLC; JLC_Part# NOT FROM JLC -> (none)
- U2: JLCPCB Part # (none) -> C16581; JLC_Part# C16581 -> (none)
- U3: JLCPCB Part # (none) -> C7955; JLC_Part# C7955 -> (none)
- U4: JLCPCB Part # (none) -> C8598; JLC_Part# C8598 -> (none)
- gave numbers to parts that had none: 2
Connections:
- net +1V5: now also TP6.1
- net +BATT: now also JP5.2 (B), TP4.1; no longer R5.1
- net LOW_BATT: now also JP2.1 (A), R12.2, TP2.1; no longer R8.1
- net VDD: now also TP1.1
- net VOUT: now also TP3.1
- net V_SW: now also JP1.1 (A), JP3.2 (B), JP4.2 (B), TP5.1; no longer C1.1, C5.2, U1.3 (VI), U3.8 (V+), U6.1 (EN), U6.4 (VIN)
- new net: JP2.2 (B), R8.1
- new net: JP5.1 (A), R5.1
- new net V+: JP3.1 (A), R12.1, U3.8 (V+)
- new net VI: C1.1, JP4.1 (A), U1.3 (VI)
- new net VIN: C5.2, JP1.2 (B), U6.1 (EN), U6.4 (VIN)
Other:
- note added: "TVS DIODE FOR ESD PROTECTION?"
- moved on the sheet: C5, C6, C7, J2, L1, R10, R11, R7, R8, R9, U4, U5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
